File: pcb/diffprobe-mainboard-v2/diffprobe-espnow.kicad_sch (KiCad schematic)
At the start: 48 parts, among them J101 Conn_01x04_Socket, J102 Conn_01x04_Socket, J103 Conn_01x04_Socket, J104 Conn_01x04_Socket, J105 Conn_01x04_Socket, J106 Conn_01x04_Socket, J107 Conn_01x04_Socket, J108 Conn_01x04_Socket, J109 Conn_01x04_Socket, J110 Conn_01x04_Socket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

Commit message: KiCAD 9 update, new psu filtering and adc input signal filtering. More silkscreen writing.
Parts:
- added H201, H202, H203, H204: MountingHole, MountingHole:MountingHole_3.2mm_M3_Pad, symbol Mechanical:MountingHole
