File: pcb/diffprobe-mainboard-v2/MagInputs.kicad_sch (KiCad schematic)
At the start: 85 parts

Commit message: schematic cleanup again
Parts:
- removed C536, C537, C538, C539, C540: ${ALTIUM_VALUE}, Capacitor_SMD:C_1206_3216Metric, symbol DifferentialProbe-altium-import:root_0_Capacitor
